File: KiCad files/LEDChristmasTree-2022/LEDChristmasTree-2022.kicad_pcb (KiCad board)
At the start: 2 copper layers, 74.9 x 92.2 mm, 0 parts

Commit message: update1
Parts:
- added BT1: Battery, Library:2xAAA-422-SMT, B.Cu at (143.6, 100.0)
- added D1: RGB, Library:LED-0807, F.Cu at (142.3, 104.4)
- added D10: RGB, Library:LED-0807, F.Cu at (129.0, 98.8)
- added D11: RGB, Library:LED-0807, F.Cu at (137.4, 76.4)
- added D2: RGB, Library:LED-0807, F.Cu at (117.2, 125.2)
- added D3: RGB, Library:LED-0807, F.Cu at (134.4, 119.4)
- added D4: RGB, Library:LED-0807, F.Cu at (144.2, 87.6)
- added D5: RGB, Library:LED-0807, F.Cu at (153.6, 116.8)
- added D6: RGB, Library:LED-0807, F.Cu at (146.4, 67.4)
- added D7: RGB, Library:LED-0807, F.Cu at (170.0, 126.6)
- added D8: RGB, Library:LED-0807, F.Cu at (157.4, 97.0)
- added D9: RGB, Library:LED-0807, F.Cu at (143.6, 51.4)
- added R1: 2k, Resistor_SMD:R_0603_1608Metric, B.Cu at (158.0, 104.4)
- added R10: 2k, Resistor_SMD:R_0603_1608Metric, B.Cu at (141.2, 66.4)
- added R11: 2k, Resistor_SMD:R_0603_1608Metric, B.Cu at (143.6, 56.8)
- added R2: 2k, Resistor_SMD:R_0603_1608Metric, B.Cu at (123.0, 125.2)
- added R3: 2k, Resistor_SMD:R_0603_1608Metric, B.Cu at (158.0, 119.4)
- added R4: 2k, Resistor_SMD:R_0603_1608Metric, B.Cu at (158.0, 94.2)
- added R5: 2k, Resistor_SMD:R_0603_1608Metric, B.Cu at (158.0, 116.8)
- added R6: 2k, Resistor_SMD:R_0603_1608Metric, B.Cu at (165.8, 126.6)
- added R7: 2k, Resistor_SMD:R_0603_1608Metric, B.Cu at (158.0, 99.8)
- added R8: 2k, Resistor_SMD:R_0603_1608Metric, B.Cu at (158.0, 92.2)
- added R9: 2k, Resistor_SMD:R_0603_1608Metric, B.Cu at (129.0, 103.4)
- added SW1: SW_SPDT, Button_Switch_SMD:SW_SPDT_PCM12, B.Cu at (171.6, 118.6)
Routing:
- net Net-(R2-Pad1): track 0.00 -> 154.0 mm
- net VCC: track 0.00 -> 29.1 mm
- net Net-(D3-Pad1): track 0.00 -> 22.9 mm, vias 0 -> 1
- net Net-(D4-Pad1): track 0.00 -> 15.8 mm, vias 0 -> 1
- net Net-(D1-Pad1): track 0.00 -> 15.4 mm, vias 0 -> 1
- net Net-(D10-Pad1): track 0.00 -> 10.3 mm, vias 0 -> 1
- net Net-(D8-Pad1): track 0.00 -> 9.41 mm, vias 0 -> 1
- net Net-(D2-Pad1): track 0.00 -> 5.07 mm, vias 0 -> 1
- net Net-(D5-Pad1): track 0.00 -> 3.67 mm, vias 0 -> 1
- net Net-(D7-Pad1): track 0.00 -> 3.47 mm, vias 0 -> 1
- net GND: vias 0 -> 4
Other:
- board size 74.9 x 92.2 mm -> 74.9 x 99.2 mm
- board text added: "JLCJLCJLCJLC"

Commit message: con
Routing:
- net unconnected-(BT1-Pad2): track 0.00 -> 51.6 mm
- net GND: vias 4 -> 0
Changed lines of the file:
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@@
   (segment (start 167.75 129.25) (end 169.8 127.2) (width 0.762) (layer "B.Cu") (net 8))
   (segment (start 149.1 129.25) (end 167.75 129.25) (width 0.762) (layer "B.Cu") (net 8))
-  (via (at 146 138) (size 0.8) (drill 0.4) (layers "F.Cu" "B.Cu") (free) (net 11))
-  (via (at 144 138) (size 0.8) (drill 0.4) (layers "F.Cu" "B.Cu") (free) (net 11))
-  (via (at 142 138) (size 0.8) (drill 0.4) (layers "F.Cu" "B.Cu") (free) (net 11))
-  (via (at 140 138) (size 0.8) (drill 0.4) (layers "F.Cu" "B.Cu") (free) (net 11))
+  (segment (start 146.2 49.3) (end 144.9 48) (width 0.762) (layer "B.Cu") (net 10))
+  (segment (start 138.1 65.4) (end 138.1 70.75) (width 0.762) (layer "B.Cu") (net 10))
+  (segment (start 146.2 63.4) (end 146.2 49.3) (width 0.762) (layer "B.Cu") (net 10))
+  (segment (start 149.1 66.3) (end 146.2 63.4) (width 0.762) (layer "B.Cu") (net 10))
+  (segment (start 149.1 70.75) (end 149.1 66.3) (width 0.762) (layer "B.Cu") (net 10))
+  (segment (start 140.8 62.7) (end 138.1 65.4) (width 0.762) (layer "B.Cu") (net 10))
+  (segment (start 140.8 49.4) (end 140.8 62.7) (width 0.762) (layer "B.Cu") (net 10))
+  (segment (start 142.2 48) (end 140.8 49.4) (width 0.762) (layer "B.Cu") (net 10))
+  (segment (start 144.9 48) (end 142.2 48) (width 0.762) (layer "B.Cu") (net 10))
   (segment (start 127.325 98.8) (end 127.95 98.175) (width 0.762) (layer "F.Cu") (net 12))
   (segment (start 126.9 98.8) (end 127.325 98.8) (width 0.762) (layer "F.Cu") (net 12))

Commit message: layout
Parts:
- moved R8 29.1 mm to (129.0, 94.4)
- moved R10 2.82 mm to (142.3, 63.8)
Routing:
- net Net-(R2-Pad1): track 154.0 -> 220.2 mm
- net Net-(D11-Pad1): track 0.00 -> 23.1 mm, vias 0 -> 1
- net unconnected-(BT1-Pad2): track 51.6 -> 45.0 mm
- net Net-(D6-Pad1): track 0.00 -> 6.28 mm, vias 0 -> 1
- net Net-(D9-Pad1): track 0.00 -> 4.67 mm, vias 0 -> 1
- net GND: vias 0 -> 20
- added copper zone on B.Cu, net GND
- added copper zone on F.Cu, net GND
