File: KiCad files/LEDChristmasTree-2022/LEDChristmasTree-2022.kicad_pcb (KiCad board)
At the start: 2 copper layers, 74.9 x 99.2 mm, 42 parts, among them SW1 SW_SPDT

Commit message: v2
Routing:
- net Net-(R1-Pad1): track 205.9 -> 0.00 mm
- net unconnected-(BT1-Pad2): track 51.9 -> 0.00 mm
- net VCC: track 31.4 -> 0.00 mm
- net Net-(D11-Pad1): track 28.0 -> 0.00 mm, vias 1 -> 0
- net Net-(D10-Pad1): track 18.0 -> 0.00 mm, vias 1 -> 0
- net Net-(D4-Pad1): track 16.7 -> 0.00 mm, vias 1 -> 0
- net Net-(D1-Pad1): track 15.9 -> 0.00 mm, vias 1 -> 0
- net Net-(D12-Pad1): track 10.9 -> 0.00 mm, vias 1 -> 0
- net Net-(D8-Pad1): track 8.23 -> 0.00 mm, vias 1 -> 0
- net Net-(D5-Pad1): track 6.17 -> 0.00 mm, vias 1 -> 0
- net Net-(D2-Pad1): track 5.02 -> 0.00 mm, vias 1 -> 0
- net Net-(D6-Pad1): track 4.83 -> 0.00 mm, vias 1 -> 0
- net Net-(D9-Pad1): track 4.67 -> 0.00 mm, vias 1 -> 0
- net Net-(D7-Pad1): track 4.47 -> 0.00 mm, vias 1 -> 0
- net Net-(D3-Pad1): track 4.44 -> 0.00 mm, vias 1 -> 0
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- removed copper zone on B.Cu, net GND
- removed copper zone on F.Cu, net GND

Commit message: v2
Parts:
- moved R1 35.7 mm to (126.0, 118.2), turned to 0 degrees
- moved R4 34.6 mm to (126.0, 104.8), turned to 0 degrees
- moved R7 33.7 mm to (126.0, 106.4), turned to 0 degrees
- moved R5 33.5 mm to (126.0, 121.4), turned to 0 degrees
- moved R6 33.5 mm to (126.0, 119.8)
- moved R8 6.62 mm to (126.0, 103.2)
- moved R12 4.45 mm to (126.0, 116.6), turned to 0 degrees
- moved R2 3.41 mm to (125.9, 124.7), turned to 0 degrees
- moved R3 3.12 mm to (125.9, 123.0)
- moved R9 2.94 mm to (126.0, 101.6), turned to 0 degrees
- moved R10 1.33 mm to (143.6, 63.5)
- moved G*** 0.76 mm to (172.7, 125.3)
- moved D7 0.10 mm to (164.7, 118.3), turned to 180 degrees
- turned D11 to 180 degrees
- turned D9 to -90 degrees
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Connections:
- net VCC renamed Net-(BT1-Pad3)
- D1 pad 1: Net-(D1-Pad1) -> GND
- D1 pad 2: GND -> Net-(D1-Pad2)
- D10 pad 1: Net-(D10-Pad1) -> GND
- D10 pad 2: GND -> Net-(D10-Pad2)
- D11 pad 1: Net-(D11-Pad1) -> GND
- D11 pad 2: GND -> Net-(D11-Pad2)
- D12 pad 1: Net-(D12-Pad1) -> GND
- D12 pad 2: GND -> Net-(D12-Pad2)
- D2 pad 1: Net-(D2-Pad1) -> GND
- D2 pad 2: GND -> Net-(D2-Pad2)
- D3 pad 1: Net-(D3-Pad1) -> GND
- D3 pad 2: GND -> Net-(D3-Pad2)
- D4 pad 1: Net-(D4-Pad1) -> GND
- D4 pad 2: GND -> Net-(D4-Pad2)
- D5 pad 1: Net-(D5-Pad1) -> GND
- D5 pad 2: GND -> Net-(D5-Pad2)
- D6 pad 1: Net-(D6-Pad1) -> GND
- D6 pad 2: GND -> Net-(D6-Pad2)
- D7 pad 1: Net-(D7-Pad1) -> GND
- D7 pad 2: GND -> Net-(D7-Pad2)
- D8 pad 1: Net-(D8-Pad1) -> GND
- D8 pad 2: GND -> Net-(D8-Pad2)
- D9 pad 1: Net-(D9-Pad1) -> GND
- D9 pad 2: GND -> Net-(D9-Pad2)
- R1 pad 2: Net-(D1-Pad1) -> Net-(D1-Pad2)
- R10 pad 2: Net-(D6-Pad1) -> Net-(D6-Pad2)
- R11 pad 2: Net-(D9-Pad1) -> Net-(D9-Pad2)
- R12 pad 2: Net-(D12-Pad1) -> Net-(D12-Pad2)
- R2 pad 2: Net-(D2-Pad1) -> Net-(D2-Pad2)
- R3 pad 2: Net-(D3-Pad1) -> Net-(D3-Pad2)
- R4 pad 2: Net-(D4-Pad1) -> Net-(D4-Pad2)
- R5 pad 2: Net-(D5-Pad1) -> Net-(D5-Pad2)
- R6 pad 2: Net-(D7-Pad1) -> Net-(D7-Pad2)
- R7 pad 2: Net-(D8-Pad1) -> Net-(D8-Pad2)
- R8 pad 2: Net-(D11-Pad1) -> Net-(D11-Pad2)
- R9 pad 2: Net-(D10-Pad1) -> Net-(D10-Pad2)
Routing:
- net Net-(R1-Pad1): track 0.00 -> 104.0 mm
- net unconnected-(BT1-Pad2): track 0.00 -> 52.2 mm
- net Net-(D7-Pad2): track 0.00 -> 38.6 mm, vias 0 -> 1
- net Net-(BT1-Pad3): track 0.00 -> 37.4 mm
- net Net-(D11-Pad2): track 0.00 -> 33.8 mm, vias 0 -> 1
- net Net-(D4-Pad2): track 0.00 -> 33.2 mm, vias 0 -> 1
- net Net-(D8-Pad2): track 0.00 -> 32.1 mm, vias 0 -> 1
- net Net-(D5-Pad2): track 0.00 -> 26.5 mm, vias 0 -> 1
- net Net-(D2-Pad2): track 0.00 -> 22.8 mm, vias 0 -> 1
- net Net-(D1-Pad2): track 0.00 -> 21.3 mm, vias 0 -> 1
- net Net-(D10-Pad2): track 0.00 -> 12.3 mm, vias 0 -> 1
- net Net-(D12-Pad2): track 0.00 -> 11.9 mm, vias 0 -> 1
- net Net-(D3-Pad2): track 0.00 -> 7.67 mm, vias 0 -> 1
- net Net-(D6-Pad2): track 0.00 -> 4.91 mm, vias 0 -> 1
- net Net-(D9-Pad2): track 0.00 -> 4.67 mm, vias 0 -> 1
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- added copper zone on B.Cu, net GND
- added copper zone on F.Cu, net GND
Other:
- board size 74.9 x 99.2 mm -> 74 x 98.1 mm
