File: KiCad files/LEDChristmasTree-2022/LEDChristmasTree-2022.kicad_sch (KiCad schematic)
At the start: 26 parts, among them SW1 SW_SPDT

Commit message: v2
Parts:
- BT1: value Battery -> (none); footprint Library:2xAAA-422-SMT -> (none)
Connections:
- net GND: now also D1.1 (K), D10.1 (K), D11.1 (K), D12.1 (K), D2.1 (K), D3.1 (K), D4.1 (K), D5.1 (K), D6.1 (K), D7.1 (K), D8.1 (K), D9.1 (K); no longer D1.2 (A), D10.2 (A), D11.2 (A), D12.2 (A), D2.2 (A), D3.2 (A), D4.2 (A), D5.2 (A), D6.2 (A), D7.2 (A), D8.2 (A), D9.2 (A)
- net at R2.2: now also D2.2 (A); no longer D2.1 (K)
- net at R3.2: now also D3.2 (A); no longer D3.1 (K)
- net at R5.2: now also D5.2 (A); no longer D5.1 (K)
- net at R7.2: now also D8.2 (A); no longer D8.1 (K)
- net at R6.2: now also D7.2 (A); no longer D7.1 (K)
- net at R8.2: now also D11.2 (A); no longer D11.1 (K)
- net at R1.2: now also D1.2 (A); no longer D1.1 (K)
- net at R10.2: now also D6.2 (A); no longer D6.1 (K)
- net at R11.2: now also D9.2 (A); no longer D9.1 (K)
- net at R4.2: now also D4.2 (A); no longer D4.1 (K)
- net at R9.2: now also D10.2 (A); no longer D10.1 (K)
- net at R12.2: now also D12.2 (A); no longer D12.1 (K)
- net VCC: no longer names the net of BT1.3 (+), SW1.1 (A)
Other:
- note added: "- naručeno 10 komada (1.2mm) pločica, cijena je 7.1kn/kom - ova narudžba je sjebana, krivi polaritet - naručeno 21 komad 2xAAA kučišta za baterije, cijena je 6,2kn/kom"
- note removed: "- naručeno 10 komada (1.2mm) pločica, cijena je 7.1kn/kom - naručeno 21 komad 2xAAA kučišta za baterije, cijena je 6,2kn/kom TODO: - zaobliti sve krakove - napraviti layout da sve ledice bude orijentirane na isti način - maknuti bijelu zvijezdu, podebljati zvijezdu bez maske"
- moved on the sheet: D1, D10, D11, D12, D2, D3, D4, D5, D6, D7, D8, D9

Commit message: images
Parts:
- BT1: value (none) -> Battery; footprint (none) -> Library:2xAAA-422-SMT
Other:
- note removed: "- naručeno 10 komada (1.2mm) pločica, cijena je 7.1kn/kom - ova narudžba je sjebana, krivi polaritet - naručeno 21 komad 2xAAA kučišta za baterije, cijena je 6,2kn/kom"
Changed lines of the file:
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@@
     (stroke (width 0) (type default) (color 0 0 0 0))
-  )
-  (text "- naručeno 10 komada (1.2mm) pločica, cijena je 7.1kn/kom - ova narudžba je sjebana, krivi polaritet\n- naručeno 21 komad 2xAAA kučišta za baterije, cijena je 6,2kn/kom "
-    (at 56.515 135.89 0)
-    (effects (font (size 2 2)) (justify left bottom))
   )
   (symbol (lib_id "Device:LED_Small") (at 111.76 81.28 90) (unit 1)
@@
       (effects (font (size 1.27 1.27)) (justify left))
     )
-    (property "Value" "" (id 1) (at 81.407 80.0612 0)
-      (effects (font (size 1.27 1.27)) (justify left))
-    )
-    (property "Footprint" "" (id 2) (at 78.74 77.216 90)
+    (property "Value" "Battery" (id 1) (at 81.407 80.0612 0)
+      (effects (font (size 1.27 1.27)) (justify left))
+    )
+    (property "Footprint" "Library:2xAAA-422-SMT" (id 2) (at 78.74 77.216 90)
       (effects (font (size 1.27 1.27)) hide)
     )
@@
       (effects (font (size 1.27 1.27)) hide)
     )
-    (property "Value" "" (id 1) (at 78.74 95.8834 0))
+    (property "Value" "GND" (id 1) (at 78.74 95.8834 0))
     (property "Footprint" "" (id 2) (at 78.74 91.44 0)
       (effects (font (size 1.27 1.27)) hide)
